Commit message: Implement frame reference to remove inertia from base_link

File: description/shippy_attachments.urdf.xacro (robot description, xacro)
@@ -48,5 +48,5 @@
       rpy="1.5707963267949 0 -1.57079632679489" />
     <parent
-      link="base_link" />
+      link="base_link_reference" />
     <child
       link="Link_Robot_Front_Attachments" />

File: description/shippy_core.urdf.xacro (robot description, xacro)
@@ -3,4 +3,12 @@
   <link
     name="base_link">
+  </link>
+  <!-- Joint connecting dummy_link to base_link -->
+  <joint name="base_link_reference" type="fixed">
+    <parent link="base_link" />
+    <child link="base_link_reference" />
+  </joint>
+  <link
+    name="base_link_reference">
     <inertial>
       <origin
@@ -88,5 +96,5 @@
       rpy="1.5707963267949 0 0" />
     <parent
-      link="base_link" />
+      link="base_link_reference" />
     <child
       link="Link_Side_Left" />
@@ -141,5 +149,5 @@
       rpy="1.5707963267949 0 0" />
     <parent
-      link="base_link" />
+      link="base_link_reference" />
     <child
       link="Link_Side_Right" />
@@ -194,5 +202,5 @@
       rpy="1.5707963267949 0 -1.57079632679489" />
     <parent
-      link="base_link" />
+      link="base_link_reference" />
     <child
       link="Link_Left_Metal" />
@@ -247,5 +255,5 @@
       rpy="1.5707963267949 0 -1.57079632679489" />
     <parent
-      link="base_link" />
+      link="base_link_reference" />
     <child
       link="Link_Right_Metal" />
@@ -300,5 +308,5 @@
       rpy="1.5707963267949 0 0" />
     <parent
-      link="base_link" />
+      link="base_link_reference" />
     <child
       link="Link_Top_Metal" />
@@ -353,5 +361,5 @@
       rpy="1.5707963267949 0 -3.14159265358979" />
     <parent
-      link="base_link" />
+      link="base_link_reference" />
     <child
       link="Link_Lackaging" />

File: description/shippy_fans.urdf.xacro (robot description, xacro)
@@ -48,5 +48,5 @@
             rpy="3.1416 -0.98049 1.5708" />
         <parent
-            link="base_link" />
+            link="base_link_reference" />
         <child
             link="Link_Left_Fan" />
@@ -101,5 +101,5 @@
             rpy="3.1416 1.2132 -1.5708" />
         <parent
-            link="base_link" />
+            link="base_link_reference" />
         <child
             link="Link_Right_Fan" />

Commit message: Adding Gazebo color tags

File: description/shippy_attachments.urdf.xacro (robot description, xacro)
@@ -41,4 +41,7 @@
     </collision>
   </link>
+  <gazebo reference="Link_Robot_Front_Attachments">
+    <material>Gazebo/ZincYellow</material>
+  </gazebo>
   <joint
     name="Joint_Robot_Front_Attachments"

File: description/shippy_core.urdf.xacro (robot description, xacro)
@@ -49,4 +49,7 @@
     </collision>
   </link>
+  <gazebo reference="base_link_reference">
+    <material>Gazebo/Green</material>
+  </gazebo>
   <link
     name="Link_Side_Left">
@@ -89,4 +92,7 @@
     </collision>
   </link>
+  <gazebo reference="Link_Side_Left">
+    <material>Gazebo/Green</material>
+  </gazebo>
   <joint
     name="Joint_Side_Left"
@@ -142,4 +148,7 @@
     </collision>
   </link>
+  <gazebo reference="Link_Side_Right">
+      <material>Gazebo/Green</material>
+  </gazebo>
   <joint
     name="Joint_Side_Right"
@@ -195,4 +204,7 @@
     </collision>
   </link>
+  <gazebo reference="Link_Left_Metal">
+    <material>Gazebo/Red</material>
+  </gazebo>
   <joint
     name="Joint_Left_Metal"
@@ -248,4 +260,7 @@
     </collision>
   </link>
+  <gazebo reference="Link_Right_Metal">
+    <material>Gazebo/Red</material>
+  </gazebo>
   <joint
     name="Joint_Right_Metal"
@@ -301,4 +316,7 @@
     </collision>
   </link>
+  <gazebo reference="Link_Top_Metal">
+    <material>Gazebo/RedBright</material>
+  </gazebo>
   <joint
     name="Joint_Top_Metal"
@@ -354,4 +372,7 @@
     </collision>
   </link>
+  <gazebo reference="Link_Lackaging">
+    <material>Gazebo/Yellow</material>
+  </gazebo>
   <joint
     name="Joint_Lackaging"

File: description/shippy_fans.urdf.xacro (robot description, xacro)
@@ -41,4 +41,7 @@
         </collision>
     </link>
+    <gazebo reference="Link_Left_Fan">
+        <material>Gazebo/Indigo</material>
+    </gazebo>
     <joint
         name="Joint_Left_Fan"
@@ -94,4 +97,7 @@
         </collision>
     </link>
+    <gazebo reference="Link_Right_Fan">
+        <material>Gazebo/Indigo</material>
+    </gazebo>
     <joint
         name="Joint_Right_Fan"
