Commit message: Edit structure to light loading and fix gazebo segmentation fault

File: description/gazebo/shippy_attachments.urdf.xacro (robot description, xacro)
@@ -2,18 +2,18 @@
 <robot xmlns:xacro="http://www.ros.org/wiki/xacro">
   <link
-    name="Link_Robot_Front_Attachments">
+    name="Link_Attach">
     <inertial>
       <origin
-        xyz="-0.110993083185633 -0.0209688861158468 -0.00942961030516409"
+        xyz="-0.00049784865130853 0.0427987016913154 0.511037262417584"
         rpy="0 0 0" />
       <mass
-        value="0.973903374699208" />
+        value="1.32876293779264" />
       <inertia
-        ixx="0.0123670881249229"
-        ixy="0.00152634507018076"
-        ixz="9.35071385864023E-07"
-        iyy="0.0163784182374264"
-        iyz="4.88372744349489E-06"
-        izz="0.00726600026096406" />
+        ixx="0.0130208817284301"
+        ixy="-4.88258049923028E-06"
+        ixz="-9.3200074052501E-07"
+        iyy="0.0225701974289401"
+        iyz="0.0015436359339137"
+        izz="0.0122028865555913" />
     </inertial>
     <visual>
@@ -23,10 +23,10 @@
       <geometry>
         <mesh
-          filename="file://$(find shippy)/meshes/Link_Robot_Front_Attachments.STL" />
+          filename="file://$(find shippy)/meshes/Link_Attach.STL" />
       </geometry>
       <material
         name="">
         <color
-          rgba="0.9 0.81 0.51 1" />
+          rgba="1 0.937254901960784 0.137254901960784 1" />
       </material>
     </visual>
@@ -37,25 +37,25 @@
       <geometry>
         <mesh
-          filename="file://$(find shippy)/meshes/Link_Robot_Front_Attachments.STL" />
+          filename="file://$(find shippy)/meshes/Link_Attach.STL" />
       </geometry>
     </collision>
   </link>
-  <gazebo reference="Link_Robot_Front_Attachments">
-    <material>Gazebo/ZincYellow</material>
-    <mu1 value="0.01"/>
-    <mu2 value="0.01"/>
-  </gazebo>
   <joint
-    name="Joint_Robot_Front_Attachments"
+    name="Joint_Attach"
     type="fixed">
     <origin
-      xyz="0 1.54252445791832 -0.10004"
-      rpy="1.5707963267949 0 -1.57079632679489" />
+      xyz="0 1.85252445791832 -0.19"
+      rpy="1.5707963267949 0 0" />
     <parent
-      link="base_link_reference" />
+      link="base_link" />
     <child
-      link="Link_Robot_Front_Attachments" />
+      link="Link_Attach" />
     <axis
       xyz="0 0 0" />
   </joint>
+  <gazebo reference="Link_Attach">
+    <material>Gazebo/ZincYellow</material>
+    <mu1 value="0.001" />
+    <mu2 value="0.001" />
+  </gazebo>
 </robot>

File: description/gazebo/shippy_core.urdf.xacro (robot description, xacro)
@@ -16,12 +16,12 @@
         rpy="0 0 0" />
       <mass
-        value="2.17957713322353" />
+        value="2.17957713322354" />
       <inertia
-        ixx="0.17899850438671"
-        ixy="5.05428036749201E-16"
-        ixz="-2.24166310386283E-16"
+        ixx="0.178998504386709"
+        ixy="5.06667889358663E-16"
+        ixz="-2.79813933858926E-16"
         iyy="0.130111023279005"
-        iyz="3.03303960572226E-05"
-        izz="0.290729649302988" />
+        iyz="3.03303960572217E-05"
+        izz="0.290729649302987" />
     </inertial>
     <visual>
@@ -50,21 +50,20 @@
   </link>
   <gazebo reference="base_link_reference">
-    <material>Gazebo/Green</material>
   </gazebo>
   <link
-    name="Link_Side_Left">
+    name="Link_SIdes">
     <inertial>
       <origin
-        xyz="0.104919265146604 0.101118372719001 0.996926007551461"
+        xyz="0.534919265146604 0.0911183727190013 0.996926007551466"
         rpy="0 0 0" />
       <mass
-        value="81.8084350434166" />
+        value="163.616870086833" />
       <inertia
-        ixx="26.245543933313"
-        ixy="-2.3094582466397E-05"
-        ixz="-0.00577226346636961"
-        iyy="26.2724801461104"
-        iyz="-0.0881450822013043"
-        izz="0.567958263795021" />
+        ixx="52.491087866626"
+        ixy="-4.61891649327673E-05"
+        ixz="-0.0115445269327401"
+        iyy="52.5449602922208"
+        iyz="-0.176290164402609"
+        izz="1.13591652759004" />
     </inertial>
     <visual>
@@ -74,5 +73,5 @@
       <geometry>
         <mesh
-          filename="file://$(find shippy)/meshes/Link_Side_Left.STL" />
+          filename="file://$(find shippy)/meshes/Link_SIdes.STL" />
       </geometry>
       <material
@@ -88,9 +87,9 @@
       <geometry>
         <mesh
-          filename="file://$(find shippy)/meshes/Link_Side_Left.STL" />
+          filename="file://$(find shippy)/meshes/Link_SIdes.STL" />
       </geometry>
     </collision>
   </link>
-  <gazebo reference="Link_Side_Left">
+  <gazebo reference="Link_SIdes">
     <material>Gazebo/Green</material>
     <mu1 value="0.0001" />
@@ -98,31 +97,31 @@
   </gazebo>
   <joint
-    name="Joint_Side_Left"
+    name="Joint_Sides"
     type="fixed">
     <origin
-      xyz="-0.535000000000017 2.01 -0.2"
+      xyz="-0.535000000000017 2.01 -0.19"
       rpy="1.5707963267949 0 0" />
     <parent
-      link="base_link_reference" />
+      link="base_link" />
     <child
-      link="Link_Side_Left" />
+      link="Link_SIdes" />
     <axis
       xyz="0 0 0" />
   </joint>
   <link
-    name="Link_Side_Right">
+    name="Link_Metal">
     <inertial>
       <origin
-        xyz="0.104919265146604 0.101118372719001 0.996926007551461"
+        xyz="0.602924866263637 0.190961400893912 -0.375"
         rpy="0 0 0" />
       <mass
-        value="81.8084350434166" />
+        value="5.54659895705767" />
       <inertia
-        ixx="26.245543933313"
-        ixy="-2.30945824663705E-05"
-        ixz="-0.00577226346637043"
-        iyy="26.2724801461104"
-        iyz="-0.0881450822013042"
-        izz="0.567958263795021" />
+        ixx="0.153378585391697"
+        ixy="-0.0237536387890743"
+        ixz="-5.04243017767317E-17"
+        iyy="0.44354732705172"
+        iyz="1.85867772292397E-17"
+        izz="0.410429972682058" />
     </inertial>
     <visual>
@@ -132,63 +131,5 @@
       <geometry>
         <mesh
-          filename="file://$(find shippy)/meshes/Link_Side_Right.STL" />
-      </geometry>
-      <material
-        name="">
-        <color
-          rgba="0.286274509803922 0.662745098039216 0.329411764705882 1" />
-      </material>
-    </visual>
-    <collision>
-      <origin
-        xyz="0 0 0"
-        rpy="0 0 0" />
-      <geometry>
-        <mesh
-          filename="file://$(find shippy)/meshes/Link_Side_Right.STL" />
-      </geometry>
-    </collision>
-  </link>
-  <gazebo reference="Link_Side_Right">
-    <material>Gazebo/Green</material>
-    <mu1 value="0.0001" />
-    <mu2 value="0.0001" />
-  </gazebo>
-  <joint
-    name="Joint_Side_Right"
-    type="fixed">
-    <origin
-      xyz="0.324999999999983 2.01 -0.2"
-      rpy="1.5707963267949 0 0" />
-    <parent
-      link="base_link_reference" />
-    <child
-      link="Link_Side_Right" />
-    <axis
-      xyz="0 0 0" />
-  </joint>
-  <link
-    name="Link_Left_Metal">
-    <inertial>
-      <origin
-        xyz="0.565954361793534 0.132380012619458 -0.0180374997719361"
-        rpy="0 0 0" />
-      <mass
-        value="1.86329947852884" />
-      <inertia
-        ixx="0.0303193760291818"
-        ixy="-0.0118768193945372"
-        ixz="-1.0311791416408E-17"
-        iyy="0.158217746859194"
-        iyz="-1.6230919151769E-17"
-        izz="0.187968319674363" />
-    </inertial>
-    <visual>
-      <origin
-        xyz="0 0 0"
-        rpy="0 0 0" />
-      <geometry>
-        <mesh
-          filename="file://$(find shippy)/meshes/Link_Left_Metal.STL" />
+          filename="file://$(find shippy)/meshes/Link_Metal.STL" />
       </geometry>
       <material
@@ -204,189 +145,21 @@
       <geometry>
         <mesh
-          filename="file://$(find shippy)/meshes/Link_Left_Metal.STL" />
+          filename="file://$(find shippy)/meshes/Link_Metal.STL" />
       </geometry>
     </collision>
   </link>
-  <gazebo reference="Link_Left_Metal">
+  <gazebo reference="Link_Metal">
     <material>Gazebo/Red</material>
   </gazebo>
   <joint
-    name="Joint_Left_Metal"
+    name="Joint_Metal"
     type="fixed">
     <origin
-      xyz="-0.375000000000015 1.76 0"
+      xyz="-0.375000000000015 1.76 0.0100000000000002"
       rpy="1.5707963267949 0 -1.57079632679489" />
     <parent
-      link="base_link_reference" />
+      link="base_link" />
     <child
-      link="Link_Left_Metal" />
-    <axis
-      xyz="0 0 0" />
-  </joint>
-  <link
-    name="Link_Right_Metal">
-    <inertial>
-      <origin
-        xyz="0.565954361793534 0.132380012619458 -0.0319625002280638"
-        rpy="0 0 0" />
-      <mass
-        value="1.86329947852884" />
-      <inertia
-        ixx="0.0303193760291818"
-        ixy="-0.0118768193945371"
-        ixz="-1.28996412691275E-18"
-        iyy="0.158217746859193"
-        iyz="-9.15073055917561E-18"
-        izz="0.187968319674362" />
-    </inertial>
-    <visual>
-      <origin
-        xyz="0 0 0"
-        rpy="0 0 0" />
-      <geometry>
-        <mesh
-          filename="file://$(find shippy)/meshes/Link_Right_Metal.STL" />
-      </geometry>
-      <material
-        name="">
-        <color
-          rgba="0.667 0.098 0.098 1" />
-      </material>
-    </visual>
-    <collision>
-      <origin
-        xyz="0 0 0"
-        rpy="0 0 0" />
-      <geometry>
-        <mesh
-          filename="file://$(find shippy)/meshes/Link_Right_Metal.STL" />
-      </geometry>
-    </collision>
-  </link>
-  <gazebo reference="Link_Right_Metal">
-    <material>Gazebo/Red</material>
-  </gazebo>
-  <joint
-    name="Joint_Right_Metal"
-    type="fixed">
-    <origin
-      xyz="0.324999999999985 1.76000000000001 0"
-      rpy="1.5707963267949 0 -1.57079632679489" />
-    <parent
-      link="base_link_reference" />
-    <child
-      link="Link_Right_Metal" />
-    <axis
-      xyz="0 0 0" />
-  </joint>
-  <link
-    name="Link_Top_Metal">
-    <inertial>
-      <origin
-        xyz="0.325 0.0100000000000001 -0.18"
-        rpy="0 0 0" />
-      <mass
-        value="1.82" />
-      <inertia
-        ixx="0.0344933333333333"
-        ixy="-4.04776950599612E-17"
-        ixz="4.26711188683265E-17"
-        iyy="0.127111833333333"
-        iyz="-1.68612496062809E-17"
-        izz="0.0927398333333331" />
-    </inertial>
-    <visual>
-      <origin
-        xyz="0 0 0"
-        rpy="0 0 0" />
-      <geometry>
-        <mesh
-          filename="file://$(find shippy)/meshes/Link_Top_Metal.STL" />
-      </geometry>
-      <material
-        name="">
-        <color
-          rgba="0.9 0.15 0.15 1" />
-      </material>
-    </visual>
-    <collision>
-      <origin
-        xyz="0 0 0"
-        rpy="0 0 0" />
-      <geometry>
-        <mesh
-          filename="file://$(find shippy)/meshes/Link_Top_Metal.STL" />
-      </geometry>
-    </collision>
-  </link>
-  <gazebo reference="Link_Top_Metal">
-    <material>Gazebo/RedBright</material>
-  </gazebo>
-  <joint
-    name="Joint_Top_Metal"
-    type="fixed">
-    <origin
-      xyz="-0.325000000000007 0.901375000000002 0.331387406397839"
-      rpy="1.5707963267949 0 0" />
-    <parent
-      link="base_link_reference" />
-    <child
-      link="Link_Top_Metal" />
-    <axis
-      xyz="0 0 0" />
-  </joint>
-  <link
-    name="Link_Lackaging">
-    <inertial>
-      <origin
-        xyz="-1.37922115839295E-07 0.000260439184406436 -0.22106537110126"
-        rpy="0 0 0" />
-      <mass
-        value="0.373244504052969" />
-      <inertia
-        ixx="0.00619580454940661"
-        ixy="-1.14148138610367E-09"
-        ixz="2.97540171867806E-09"
-        iyy="0.00619819616642874"
-        iyz="-1.72909730673878E-05"
-        izz="0.000270307716248751" />
-    </inertial>
-    <visual>
-      <origin
-        xyz="0 0 0"
-        rpy="0 0 0" />
-      <geometry>
-        <mesh
-          filename="file://$(find shippy)/meshes/Link_Lackaging.STL" />
-      </geometry>
-      <material
-        name="">
-        <color
-          rgba="1 0.937254901960784 0.137254901960784 1" />
-      </material>
-    </visual>
-    <collision>
-      <origin
-        xyz="0 0 0"
-        rpy="0 0 0" />
-      <geometry>
-        <mesh
-          filename="file://$(find shippy)/meshes/Link_Lackaging.STL" />
-      </geometry>
-    </collision>
-  </link>
-  <gazebo reference="Link_Lackaging">
-    <material>Gazebo/Yellow</material>
-  </gazebo>
-  <joint
-    name="Joint_Lackaging"
-    type="fixed">
-    <origin
-      xyz="0 0.702000000000005 -0.0100000000000001"
-      rpy="1.5707963267949 0 -3.14159265358979" />
-    <parent
-      link="base_link_reference" />
-    <child
-      link="Link_Lackaging" />
+      link="Link_Metal" />
     <axis
       xyz="0 0 0" />
