Commit message: Update lidar postion and visualization and gazebo colors of robot

File: description/gazebo/lidar.xacro (robot description, xacro)
@@ -4,5 +4,5 @@
         <parent link="base_link" />
         <child link="laser_frame" />
-        <origin xyz="0 1.07 0.375" rpy="0 0 0" />
+        <origin xyz="1.07 0 0.375" rpy="0 0 0" />
     </joint>
     <link name="laser_frame">
@@ -25,5 +25,5 @@
         <sensor name="laser" type="ray">
             <pose> 0 0 0 0 0 0 </pose>
-            <visualize>true</visualize>
+            <visualize>false</visualize>
             <update_rate>10</update_rate>
             <ray>

File: description/gazebo/shippy_collision.xacro (robot description, xacro)
@@ -48,4 +48,12 @@
     <link name="base_link">
     </link>
+    <!-- BASE LINK -->
+    <joint name="base_footprint_joint" type="fixed">
+        <parent link="base_link" />
+        <child link="base_footprint" />
+        <origin xyz="0 0 0" rpy="0 0 0" />
+    </joint>
+    <link name="base_footprint">
+    </link>
     <!-- CHASSIS LINK -->
     <joint name="chassis_joint" type="fixed">
@@ -90,4 +98,7 @@
         </xacro:inertial_cylinder>
     </link>
+    <gazebo reference="left_wheel">
+        <material>Gazebo/Orange</material>
+    </gazebo>
     <!-- RIGHT WHEEL LINK -->
     <joint name="Joint_Right_Fan" type="continuous">
@@ -112,5 +123,5 @@
     </link>
     <gazebo reference="right_wheel">
-        <material>Gazebo/Blue</material>
+        <material>Gazebo/Orange</material>
     </gazebo>
     <!-- CASTER WHEEL LINK -->

File: description/gazebo/shippy_visual.xacro (robot description, xacro)
@@ -31,4 +31,5 @@
     </link>
     <gazebo reference="base_link_reference">
+        <material>Gazebo/White</material>
     </gazebo>
     <!-- ! Green Sides -->
@@ -55,5 +56,5 @@
         </visual>
     </link>
-    <gazebo reference="Link_SIdes">
+    <gazebo reference="link_visual_sides">
         <material>Gazebo/Green</material>
     </gazebo>
@@ -103,5 +104,5 @@
         </visual>
     </link>
-    <gazebo reference="Link_Attach">
+    <gazebo reference="link_visual_attach">
         <material>Gazebo/ZincYellow</material>
     </gazebo>
