Commit message: Add launch robot with edit on ros2_control and yaml file ; && Save rviz

File: description/gazebo/ros2_control.xacro (robot description, xacro)
@@ -1,5 +1,33 @@
 <?xml version="1.0"?>
 <robot xmlns:xacro="http://www.ros.org/wiki/xacro">
-    <ros2_control name="GazeboSystem" type="system">
+    <ros2_control name="RealRobot" type="system">
+        <hardware>
+            <plugin>diffdrive_arduino/DiffDriveArduino</plugin>
+            <param name="left_wheel_name">Joint_Left_Fan</param>
+            <param name="right_wheel_name">Joint_Right_Fan</param>
+            <param name="loop_rate">30</param>
+            <param name="device">/dev/serial/by-path/platform-fd500000.pcie-pci-0000:01:00.0-usb-0:1.3:1.0-port0</param>
+            <param name="baud_rate">57600</param>
+            <param name="timeout">1000</param>
+            <param name="enc_counts_per_rev">3436</param>
+        </hardware>
+        <joint name="Joint_Left_Fan">
+            <command_interface name="velocity">
+                <param name="min">-10.0</param>
+                <param name="max">10.0</param>
+            </command_interface>
+            <state_interface name="velocity" />
+            <state_interface name="position" />
+        </joint>
+        <joint name="Joint_Right_Fan">
+            <command_interface name="velocity">
+                <param name="min">-10.0</param>
+                <param name="max">10.0</param>
+            </command_interface>
+            <state_interface name="velocity" />
+            <state_interface name="position" />
+        </joint>
+    </ros2_control>
+    <!-- <ros2_control name="GazeboSystem" type="system">
         <hardware>
             <plugin>gazebo_ros2_control/GazeboSystem</plugin>
@@ -21,5 +49,5 @@
             <state_interface name="position" />
         </joint>
-    </ros2_control>
+    </ros2_control> -->
     <gazebo>
         <plugin name="gazebo_ros2_control" filename="libgazebo_ros2_control.so">

Commit message: Add swtich between real robot and simulation using sim_mode

File: description/gazebo/ros2_control.xacro (robot description, xacro)
@@ -1,56 +1,61 @@
 <?xml version="1.0"?>
 <robot xmlns:xacro="http://www.ros.org/wiki/xacro">
-    <ros2_control name="RealRobot" type="system">
-        <hardware>
-            <plugin>diffdrive_arduino/DiffDriveArduino</plugin>
-            <param name="left_wheel_name">Joint_Left_Fan</param>
-            <param name="right_wheel_name">Joint_Right_Fan</param>
-            <param name="loop_rate">30</param>
-            <param name="device">/dev/serial/by-path/platform-fd500000.pcie-pci-0000:01:00.0-usb-0:1.3:1.0-port0</param>
-            <param name="baud_rate">57600</param>
-            <param name="timeout">1000</param>
-            <param name="enc_counts_per_rev">3436</param>
-        </hardware>
-        <joint name="Joint_Left_Fan">
-            <command_interface name="velocity">
-                <param name="min">-10.0</param>
-                <param name="max">10.0</param>
-            </command_interface>
-            <state_interface name="velocity" />
-            <state_interface name="position" />
-        </joint>
-        <joint name="Joint_Right_Fan">
-            <command_interface name="velocity">
-                <param name="min">-10.0</param>
-                <param name="max">10.0</param>
-            </command_interface>
-            <state_interface name="velocity" />
-            <state_interface name="position" />
-        </joint>
-    </ros2_control>
-    <!-- <ros2_control name="GazeboSystem" type="system">
-        <hardware>
-            <plugin>gazebo_ros2_control/GazeboSystem</plugin>
-        </hardware>
-        <joint name="Joint_Left_Fan">
-            <command_interface name="velocity">
-                <param name="min">-10.0</param>
-                <param name="max">10.0</param>
-            </command_interface>
-            <state_interface name="velocity" />
-            <state_interface name="position" />
-        </joint>
-        <joint name="Joint_Right_Fan">
-            <command_interface name="velocity">
-                <param name="min">-10.0</param>
-                <param name="max">10.0</param>
-            </command_interface>
-            <state_interface name="velocity" />
-            <state_interface name="position" />
-        </joint>
-    </ros2_control> -->
+    <xacro:unless value="$(arg sim_mode)">
+        <ros2_control name="RealRobot" type="system">
+            <hardware>
+                <plugin>diffdrive_arduino/DiffDriveArduino</plugin>
+                <param name="left_wheel_name">Joint_Left_Fan</param>
+                <param name="right_wheel_name">Joint_Right_Fan</param>
+                <param name="loop_rate">30</param>
+                <param name="device">/dev/serial/by-path/platform-fd500000.pcie-pci-0000:01:00.0-usb-0:1.3:1.0-port0</param>
+                <param name="baud_rate">57600</param>
+                <param name="timeout">1000</param>
+                <param name="enc_counts_per_rev">3436</param>
+            </hardware>
+            <joint name="Joint_Left_Fan">
+                <command_interface name="velocity">
+                    <param name="min">-10.0</param>
+                    <param name="max">10.0</param>
+                </command_interface>
+                <state_interface name="velocity" />
+                <state_interface name="position" />
+            </joint>
+            <joint name="Joint_Right_Fan">
+                <command_interface name="velocity">
+                    <param name="min">-10.0</param>
+                    <param name="max">10.0</param>
+                </command_interface>
+                <state_interface name="velocity" />
+                <state_interface name="position" />
+            </joint>
+        </ros2_control>
+    </xacro:unless>
+    <xacro:if value="$(arg sim_mode)">
+        <ros2_control name="GazeboSystem" type="system">
+            <hardware>
+                <plugin>gazebo_ros2_control/GazeboSystem</plugin>
+            </hardware>
+            <joint name="Joint_Left_Fan">
+                <command_interface name="velocity">
+                    <param name="min">-10.0</param>
+                    <param name="max">10.0</param>
+                </command_interface>
+                <state_interface name="velocity" />
+                <state_interface name="position" />
+            </joint>
+            <joint name="Joint_Right_Fan">
+                <command_interface name="velocity">
+                    <param name="min">-10.0</param>
+                    <param name="max">10.0</param>
+                </command_interface>
+                <state_interface name="velocity" />
+                <state_interface name="position" />
+            </joint>
+        </ros2_control>
+    </xacro:if>
     <gazebo>
         <plugin name="gazebo_ros2_control" filename="libgazebo_ros2_control.so">
             <parameters>$(find shippy)/config/my_controllers.yaml</parameters>
+            <parameters>$(find shippy)/config/gaz_ros2_ctl_use_sim.yaml</parameters>
         </plugin>
     </gazebo>

File: description/gazebo/shippy.urdf.xacro (robot description, xacro)
@@ -2,4 +2,5 @@
 <robot xmlns:xacro="http://www.ros.org/wiki/xacro" name="Shippy">
   <xacro:arg name="use_ros2_control" default="true"/>
+  <xacro:arg name="sim_mode" default="false"/>
   <xacro:if value="$(arg use_ros2_control)">
       <xacro:include filename="ros2_control.xacro" />
